Commit message: Added mock joint interfaces to urdf and test server

File: opcua_bringup/urdf/control/opcua_macro.ros2_control.xacro (robot description, xacro)
@@ -43,14 +43,12 @@
             <gpio name="robot_command">
                 <xacro:command_interface_OPCUA name="my_integer_interface" data_type="double" ua_type="UA_Int32" ua_ns="1" ua_identifier="1" initial_value="42.0"/>
-                 <xacro:command_interface_OPCUA name="commandPos_0" data_type="double" ua_type="UA_Boolean" ua_ns="1" ua_identifier="11" n_elements="2" index="0" initial_value="0"/>
+                <xacro:command_interface_OPCUA name="commandPos_0" data_type="double" ua_type="UA_Boolean" ua_ns="1" ua_identifier="11" n_elements="2" index="0" initial_value="0"/>
                 <xacro:command_interface_OPCUA name="commandPos_1" data_type="double" ua_type="UA_Boolean" ua_ns="1" ua_identifier="11" n_elements="2" index="1" initial_value="1"/>
             </gpio>
-            <!-- <gpio name="gripper">
-                <xacro:command_interface_OPCUA name="close" data_type="bool" ua_type="bool" ua_ns="4" ua_identifier="19" initial_value="true"/>
-                <xacro:command_interface_OPCUA name="open" data_type="bool" ua_type="bool" ua_ns="4" ua_identifier="20" initial_value="false"/>
-            </gpio>
-            <sensor name="gripper_sensor">
-                <xacro:state_interface_OPCUA name="object_sensor" data_type="bool" ua_type="bool" ua_ns="4" ua_identifier="109" initial_value="true"/>
-            </sensor> -->
+            <joint name="mock_joint">
+                <xacro:command_interface_OPCUA name="velocity" data_type="double" ua_type="UA_Double" ua_ns="1" ua_identifier="4" unit="mm/s" min="0" max="500"/>
+                <xacro:state_interface_OPCUA name="velocity" data_type="double" ua_type="UA_Double" ua_ns="1" ua_identifier="4" unit="mm/s" min="0" max="500" />
+                <xacro:state_interface_OPCUA name="position" data_type="double" ua_type="UA_Double" ua_ns="1" ua_identifier="5" unit="mm" min="0" max="200"/>
+            </joint>
         </ros2_control>
     </xacro:macro>

File: opcua_bringup/urdf/opcua.urdf.xacro (robot description, xacro)
@@ -10,4 +10,11 @@
   <!-- create link fixed to the "world" -->
   <link name="world"/>
+  <link name="mock_link"/>
+  <joint name="mock_passive_joint" type="continuous">
+    <parent link="world"/>
+    <child link="mock_link"/>
+    <origin xyz="0 0 0" rpy="0 0 0"/>
+    <axis xyz="0 0 1"/>
+  </joint>
   <xacro:opcua_ros2_control
     name="opcua_bot"
