Commit message: Read and set value of a state interface from the UA server

File: opcua_bringup/urdf/control/opcua_interfaces.ros2_control.xacro (robot description, xacro)
@@ -11,6 +11,6 @@
         </command_interface>
     </xacro:macro>
-    <xacro:macro name="state_interface_OPCUA" params="name data_type ua_type ua_ns ua_identifier initial_value:=0">
-        <state_interface name="${name}" data_type="${data_type}">
+    <xacro:macro name="state_interface_OPCUA" params="name ua_type ua_ns ua_identifier initial_value:=0">
+        <state_interface name="${name}">
             <xacro:if value="${initial_value != ''}">
                 <param name="initial_value">${initial_value}</param>

File: opcua_bringup/urdf/control/opcua_macro.ros2_control.xacro (robot description, xacro)
@@ -21,5 +21,5 @@
             </hardware>
             <!-- These interfaces can be declared for any component - joint, gpio or sensor -->
-            <gpio name="gripper">
+            <!-- <gpio name="gripper">
                 <xacro:command_interface_OPCUA name="close" data_type="bool" ua_type="bool" ua_ns="4" ua_identifier="19" initial_value="true"/>
                 <xacro:command_interface_OPCUA name="cose" data_type="bool" ua_type="bool" ua_ns="4" ua_identifier="20" initial_value="false"/>
@@ -27,4 +27,7 @@
             <sensor name="gripper_sensor">
                 <xacro:state_interface_OPCUA name="object_sensor" data_type="bool" ua_type="bool" ua_ns="4" ua_identifier="109" initial_value="true"/>
+            </sensor> -->
+             <sensor name="my_integer">
+                <xacro:state_interface_OPCUA name="my_integer_interface" ua_type="UA_Int32" ua_ns="1" ua_identifier="1"/>
             </sensor>
         </ros2_control>

Commit message: Write value to UA server for a single command interface

File: opcua_bringup/urdf/control/opcua_interfaces.ros2_control.xacro (robot description, xacro)
@@ -11,6 +11,6 @@
         </command_interface>
     </xacro:macro>
-    <xacro:macro name="state_interface_OPCUA" params="name ua_type ua_ns ua_identifier initial_value:=0">
-        <state_interface name="${name}">
+    <xacro:macro name="state_interface_OPCUA" params="name data_type ua_type ua_ns ua_identifier initial_value:=0">
+        <state_interface name="${name}" data_type="${data_type}">
             <xacro:if value="${initial_value != ''}">
                 <param name="initial_value">${initial_value}</param>

File: opcua_bringup/urdf/control/opcua_macro.ros2_control.xacro (robot description, xacro)
@@ -23,12 +23,16 @@
             <!-- <gpio name="gripper">
                 <xacro:command_interface_OPCUA name="close" data_type="bool" ua_type="bool" ua_ns="4" ua_identifier="19" initial_value="true"/>
-                <xacro:command_interface_OPCUA name="cose" data_type="bool" ua_type="bool" ua_ns="4" ua_identifier="20" initial_value="false"/>
+                <xacro:command_interface_OPCUA name="open" data_type="bool" ua_type="bool" ua_ns="4" ua_identifier="20" initial_value="false"/>
             </gpio>
             <sensor name="gripper_sensor">
                 <xacro:state_interface_OPCUA name="object_sensor" data_type="bool" ua_type="bool" ua_ns="4" ua_identifier="109" initial_value="true"/>
             </sensor> -->
-             <sensor name="my_integer">
-                <xacro:state_interface_OPCUA name="my_integer_interface" ua_type="UA_Int32" ua_ns="1" ua_identifier="1"/>
+             <sensor name="my_integer_sensor">
+                <!-- <xacro:state_interface_OPCUA name="my_integer_interface" data_type="uint32" ua_type="UA_Int32" ua_ns="1" ua_identifier="1"/>    -->
+                <xacro:state_interface_OPCUA name="my_integer_interface" data_type="double" ua_type="UA_Int32" ua_ns="1" ua_identifier="1"/>
             </sensor>
+            <!-- <gpio name="my_integer_command"> -->
+                <!-- <xacro:command_interface_OPCUA name="my_integer_interface" data_type="double" ua_type="UA_Int32" ua_ns="1" ua_identifier="1" initial_value="42.0"/>  -->
+            <!-- </gpio> -->
         </ros2_control>
     </xacro:macro>

Commit message: Implemented read operation for state interfaces of type ARRAY[x]

File: opcua_bringup/urdf/control/opcua_interfaces.ros2_control.xacro (robot description, xacro)
@@ -1,5 +1,5 @@
 <?xml version="1.0" encoding="UTF-8"?>
 <robot xmlns:xacro="http://wiki.ros.org/xacro">
-    <xacro:macro name="command_interface_OPCUA" params="name data_type ua_type ua_ns ua_identifier initial_value:=0">
+    <xacro:macro name="command_interface_OPCUA" params="name data_type ua_type ua_ns ua_identifier n_elements:=1 index:='' initial_value:=0">
         <command_interface name="${name}" data_type="${data_type}">
             <xacro:if value="${initial_value != ''}">
@@ -9,7 +9,11 @@
             <param name="ua_ns">${ua_ns}</param>
             <param name="ua_identifier">${ua_identifier}</param>
+            <param name="n_elements">${n_elements}</param>
+            <xacro:if value="${index != ''}">
+                <param name="index">${index}</param>
+            </xacro:if>
         </command_interface>
     </xacro:macro>
-    <xacro:macro name="state_interface_OPCUA" params="name data_type ua_type ua_ns ua_identifier initial_value:=0">
+    <xacro:macro name="state_interface_OPCUA" params="name data_type ua_type ua_ns ua_identifier n_elements:=1 index:='' initial_value:=0">
         <state_interface name="${name}" data_type="${data_type}">
             <xacro:if value="${initial_value != ''}">
@@ -19,4 +23,8 @@
             <param name="ua_ns">${ua_ns}</param>
             <param name="ua_identifier">${ua_identifier}</param>
+            <param name="n_elements">${n_elements}</param>
+            <xacro:if value="${index != ''}">
+                <param name="index">${index}</param>
+            </xacro:if>
         </state_interface>
     </xacro:macro>

File: opcua_bringup/urdf/control/opcua_macro.ros2_control.xacro (robot description, xacro)
@@ -21,4 +21,13 @@
             </hardware>
             <!-- These interfaces can be declared for any component - joint, gpio or sensor -->
+            <!-- IMPORTANT With the current implementation the indexes of same Array SHOULD be ordered in an ascending manner and declared consecutively -->
+            <sensor name="robot_sensor">
+                <xacro:state_interface_OPCUA name="my_integer_interface" data_type="double" ua_type="UA_Int32" ua_ns="1" ua_identifier="1"/>
+                <xacro:state_interface_OPCUA name="currentPos_0" data_type="double" ua_type="UA_Float" ua_ns="1" ua_identifier="10" n_elements="2" index="0"/>
+                <xacro:state_interface_OPCUA name="currentPos_1" data_type="double" ua_type="UA_Float" ua_ns="1" ua_identifier="10" n_elements="2" index="1"/>
+            </sensor>
+            <gpio name="my_integer_command">
+                <xacro:command_interface_OPCUA name="my_integer_interface" data_type="double" ua_type="UA_Int32" ua_ns="1" ua_identifier="1" initial_value="42.0"/>
+            </gpio>
             <!-- <gpio name="gripper">
                 <xacro:command_interface_OPCUA name="close" data_type="bool" ua_type="bool" ua_ns="4" ua_identifier="19" initial_value="true"/>
@@ -28,11 +37,4 @@
                 <xacro:state_interface_OPCUA name="object_sensor" data_type="bool" ua_type="bool" ua_ns="4" ua_identifier="109" initial_value="true"/>
             </sensor> -->
-             <sensor name="my_integer_sensor">
-                <!-- <xacro:state_interface_OPCUA name="my_integer_interface" data_type="uint32" ua_type="UA_Int32" ua_ns="1" ua_identifier="1"/>    -->
-                <xacro:state_interface_OPCUA name="my_integer_interface" data_type="double" ua_type="UA_Int32" ua_ns="1" ua_identifier="1"/>
-            </sensor>
-            <gpio name="my_integer_command">
-                <xacro:command_interface_OPCUA name="my_integer_interface" data_type="double" ua_type="UA_Int32" ua_ns="1" ua_identifier="1" initial_value="42.0"/>
-            </gpio>
         </ros2_control>
     </xacro:macro>

Commit message: Add parameters to state/command interfaces macro

File: opcua_bringup/urdf/control/opcua_interfaces.ros2_control.xacro (robot description, xacro)
@@ -1,5 +1,5 @@
 <?xml version="1.0" encoding="UTF-8"?>
 <robot xmlns:xacro="http://wiki.ros.org/xacro">
-    <xacro:macro name="command_interface_OPCUA" params="name data_type ua_type ua_ns ua_identifier n_elements:=1 index:='' initial_value:=0">
+    <xacro:macro name="command_interface_OPCUA" params="name data_type ua_type ua_ns ua_identifier unit min max scaling_factor n_elements:=1 index:='' initial_value:=0">
         <command_interface name="${name}" data_type="${data_type}">
             <xacro:if value="${initial_value != ''}">
@@ -9,4 +9,8 @@
             <param name="ua_ns">${ua_ns}</param>
             <param name="ua_identifier">${ua_identifier}</param>
+            <param name="unit">${unit}</param>
+            <param name="min">${min}</param>
+            <param name="max">${max}</param>
+            <param name="scaling_factor">${scaling_factor}</param>
             <param name="n_elements">${n_elements}</param>
             <xacro:if value="${index != ''}">
@@ -15,5 +19,5 @@
         </command_interface>
     </xacro:macro>
-    <xacro:macro name="state_interface_OPCUA" params="name data_type ua_type ua_ns ua_identifier n_elements:=1 index:='' initial_value:=0">
+    <xacro:macro name="state_interface_OPCUA" params="name data_type ua_type ua_ns ua_identifier unit min max scaling_factor n_elements:=1 index:='' initial_value:=0">
         <state_interface name="${name}" data_type="${data_type}">
             <xacro:if value="${initial_value != ''}">
@@ -23,4 +27,8 @@
             <param name="ua_ns">${ua_ns}</param>
             <param name="ua_identifier">${ua_identifier}</param>
+            <param name="unit">${unit}</param>
+            <param name="min">${min}</param>
+            <param name="max">${max}</param>
+            <param name="scaling_factor">${scaling_factor}</param>
             <param name="n_elements">${n_elements}</param>
             <xacro:if value="${index != ''}">

Commit message: Make the unit/max/min/scaling_factor params optional

File: opcua_bringup/urdf/control/opcua_interfaces.ros2_control.xacro (robot description, xacro)
@@ -1,5 +1,5 @@
 <?xml version="1.0" encoding="UTF-8"?>
 <robot xmlns:xacro="http://wiki.ros.org/xacro">
-    <xacro:macro name="command_interface_OPCUA" params="name data_type ua_type ua_ns ua_identifier unit min max scaling_factor n_elements:=1 index:='' initial_value:=0">
+    <xacro:macro name="command_interface_OPCUA" params="name data_type ua_type ua_ns ua_identifier unit:='' min:='' max:=''' scaling_factor:='' n_elements:=1 index:='' initial_value:=0">
         <command_interface name="${name}" data_type="${data_type}">
             <xacro:if value="${initial_value != ''}">
@@ -9,9 +9,17 @@
             <param name="ua_ns">${ua_ns}</param>
             <param name="ua_identifier">${ua_identifier}</param>
-            <param name="unit">${unit}</param>
-            <param name="min">${min}</param>
-            <param name="max">${max}</param>
-            <param name="scaling_factor">${scaling_factor}</param>
             <param name="n_elements">${n_elements}</param>
+            <xacro:if value="${unit != ''}">
+                <param name="unit">${unit}</param>
+            </xacro:if>
+             <xacro:if value="${min != ''}">
+                <param name="min">${min}</param>
+            </xacro:if>
+            <xacro:if value="${max != ''}">
+                <param name="max">${max}</param>
+            </xacro:if>
+            <xacro:if value="${scaling_factor != ''}">
+                <param name="scaling_factor">${scaling_factor}</param>
+            </xacro:if>
             <xacro:if value="${index != ''}">
                 <param name="index">${index}</param>
@@ -19,5 +27,5 @@
         </command_interface>
     </xacro:macro>
-    <xacro:macro name="state_interface_OPCUA" params="name data_type ua_type ua_ns ua_identifier unit min max scaling_factor n_elements:=1 index:='' initial_value:=0">
+    <xacro:macro name="state_interface_OPCUA" params="name data_type ua_type ua_ns ua_identifier unit:='' min:='' max:='' scaling_factor:='' n_elements:=1 index:='' initial_value:=0">
         <state_interface name="${name}" data_type="${data_type}">
             <xacro:if value="${initial_value != ''}">
@@ -27,9 +35,17 @@
             <param name="ua_ns">${ua_ns}</param>
             <param name="ua_identifier">${ua_identifier}</param>
-            <param name="unit">${unit}</param>
-            <param name="min">${min}</param>
-            <param name="max">${max}</param>
-            <param name="scaling_factor">${scaling_factor}</param>
             <param name="n_elements">${n_elements}</param>
+            <xacro:if value="${unit != ''}">
+                <param name="unit">${unit}</param>
+            </xacro:if>
+             <xacro:if value="${min != ''}">
+                <param name="min">${min}</param>
+            </xacro:if>
+            <xacro:if value="${max != ''}">
+                <param name="max">${max}</param>
+            </xacro:if>
+            <xacro:if value="${scaling_factor != ''}">
+                <param name="scaling_factor">${scaling_factor}</param>
+            </xacro:if>
             <xacro:if value="${index != ''}">
                 <param name="index">${index}</param>

Commit message: Fix min max params override
min/max are native parameters so we replace ours with min_val/max_val

File: opcua_bringup/urdf/control/opcua_interfaces.ros2_control.xacro (robot description, xacro)
@@ -1,5 +1,5 @@
 <?xml version="1.0" encoding="UTF-8"?>
 <robot xmlns:xacro="http://wiki.ros.org/xacro">
-    <xacro:macro name="command_interface_OPCUA" params="name data_type ua_type ua_ns ua_identifier unit:='' min:='' max:=''' scaling_factor:='' n_elements:=1 index:='' initial_value:=0">
+    <xacro:macro name="command_interface_OPCUA" params="name data_type ua_type ua_ns ua_identifier unit:='' min_val:='' max_val:='' scaling_factor:='' n_elements:=1 index:='' initial_value:=0">
         <command_interface name="${name}" data_type="${data_type}">
             <xacro:if value="${initial_value != ''}">
@@ -13,9 +13,9 @@
                 <param name="unit">${unit}</param>
             </xacro:if>
-             <xacro:if value="${min != ''}">
-                <param name="min">${min}</param>
+             <xacro:if value="${min_val != ''}">
+                <param name="min">${min_val}</param>
             </xacro:if>
-            <xacro:if value="${max != ''}">
-                <param name="max">${max}</param>
+            <xacro:if value="${max_val != ''}">
+                <param name="max">${max_val}</param>
             </xacro:if>
             <xacro:if value="${scaling_factor != ''}">
@@ -27,5 +27,5 @@
         </command_interface>
     </xacro:macro>
-    <xacro:macro name="state_interface_OPCUA" params="name data_type ua_type ua_ns ua_identifier unit:='' min:='' max:='' scaling_factor:='' n_elements:=1 index:='' initial_value:=0">
+    <xacro:macro name="state_interface_OPCUA" params="name data_type ua_type ua_ns ua_identifier unit:='' min_val:='' max_val:='' scaling_factor:='' n_elements:=1 index:='' initial_value:=0">
         <state_interface name="${name}" data_type="${data_type}">
             <xacro:if value="${initial_value != ''}">
@@ -39,9 +39,9 @@
                 <param name="unit">${unit}</param>
             </xacro:if>
-             <xacro:if value="${min != ''}">
-                <param name="min">${min}</param>
+             <xacro:if value="${min_val != ''}">
+                <param name="min">${min_val}</param>
             </xacro:if>
-            <xacro:if value="${max != ''}">
-                <param name="max">${max}</param>
+            <xacro:if value="${max_val != ''}">
+                <param name="max">${max_val}</param>
             </xacro:if>
             <xacro:if value="${scaling_factor != ''}">

File: opcua_bringup/urdf/control/opcua_macro.ros2_control.xacro (robot description, xacro)
@@ -47,7 +47,7 @@
             </gpio>
             <joint name="mock_joint">
-                <xacro:command_interface_OPCUA name="velocity" data_type="double" ua_type="UA_Double" ua_ns="1" ua_identifier="4" unit="mm/s" min="0" max="500"/>
-                <xacro:state_interface_OPCUA name="velocity" data_type="double" ua_type="UA_Double" ua_ns="1" ua_identifier="4" unit="mm/s" min="0" max="500" />
-                <xacro:state_interface_OPCUA name="position" data_type="double" ua_type="UA_Double" ua_ns="1" ua_identifier="5" unit="mm" min="0" max="200"/>
+                <xacro:command_interface_OPCUA name="velocity" data_type="double" ua_type="UA_Double" ua_ns="1" ua_identifier="4" unit="mm/s" min_val="0.0" max_val="500.0"/>
+                <xacro:state_interface_OPCUA name="velocity" data_type="double" ua_type="UA_Double" ua_ns="1" ua_identifier="4" unit="mm/s" min_val="0.0" max_val="500.0"/>
+                <xacro:state_interface_OPCUA name="position" data_type="double" ua_type="UA_Double" ua_ns="1" ua_identifier="5" unit="mm" min_val="0.0" max_val="100.0"/>
             </joint>
         </ros2_control>

Commit message: Remove unit parameter from URDF and hardware interface

File: opcua_bringup/urdf/control/opcua_interfaces.ros2_control.xacro (robot description, xacro)
@@ -1,5 +1,5 @@
 <?xml version="1.0" encoding="UTF-8"?>
 <robot xmlns:xacro="http://wiki.ros.org/xacro">
-    <xacro:macro name="command_interface_OPCUA" params="name data_type ua_type ua_ns ua_identifier unit:='' min_val:='' max_val:='' scaling_factor:='' n_elements:=1 index:='' initial_value:=0">
+    <xacro:macro name="command_interface_OPCUA" params="name data_type ua_type ua_ns ua_identifier min_val:='' max_val:='' scaling_factor:='' n_elements:=1 index:='' initial_value:=0">
         <command_interface name="${name}" data_type="${data_type}">
             <xacro:if value="${initial_value != ''}">
@@ -10,7 +10,4 @@
             <param name="ua_identifier">${ua_identifier}</param>
             <param name="n_elements">${n_elements}</param>
-            <xacro:if value="${unit != ''}">
-                <param name="unit">${unit}</param>
-            </xacro:if>
              <xacro:if value="${min_val != ''}">
                 <param name="min">${min_val}</param>
@@ -27,5 +24,5 @@
         </command_interface>
     </xacro:macro>
-    <xacro:macro name="state_interface_OPCUA" params="name data_type ua_type ua_ns ua_identifier unit:='' min_val:='' max_val:='' scaling_factor:='' n_elements:=1 index:='' initial_value:=0">
+    <xacro:macro name="state_interface_OPCUA" params="name data_type ua_type ua_ns ua_identifier min_val:='' max_val:='' scaling_factor:='' n_elements:=1 index:='' initial_value:=0">
         <state_interface name="${name}" data_type="${data_type}">
             <xacro:if value="${initial_value != ''}">
@@ -36,7 +33,4 @@
             <param name="ua_identifier">${ua_identifier}</param>
             <param name="n_elements">${n_elements}</param>
-            <xacro:if value="${unit != ''}">
-                <param name="unit">${unit}</param>
-            </xacro:if>
              <xacro:if value="${min_val != ''}">
                 <param name="min">${min_val}</param>

File: opcua_bringup/urdf/control/opcua_macro.ros2_control.xacro (robot description, xacro)
@@ -47,7 +47,7 @@
             </gpio>
             <joint name="mock_joint">
-                <xacro:command_interface_OPCUA name="velocity" data_type="double" ua_type="UA_Double" ua_ns="1" ua_identifier="4" unit="mm/s" min_val="0.0" max_val="500.0"/>
-                <xacro:state_interface_OPCUA name="velocity" data_type="double" ua_type="UA_Double" ua_ns="1" ua_identifier="4" unit="mm/s" min_val="0.0" max_val="500.0"/>
-                <xacro:state_interface_OPCUA name="position" data_type="double" ua_type="UA_Double" ua_ns="1" ua_identifier="5" unit="mm" min_val="0.0" max_val="100.0"/>
+                <xacro:command_interface_OPCUA name="velocity" data_type="double" ua_type="UA_Double" ua_ns="1" ua_identifier="4" min_val="-0.5" max_val="0.5"/>
+                <xacro:state_interface_OPCUA name="velocity" data_type="double" ua_type="UA_Double" ua_ns="1" ua_identifier="4" min_val="-0.5" max_val="0.5"/>
+                <xacro:state_interface_OPCUA name="position" data_type="double" ua_type="UA_Double" ua_ns="1" ua_identifier="5" min_val="0.0" max_val="0.2"/>
             </joint>
         </ros2_control>
